Commit message: 11_13: controller, slam_toolbox

File: description/robot.urdf.xacro (robot description, xacro)
@@ -2,4 +2,6 @@
 <robot xmlns:xacro="http://www.ros.org/wiki/xacro"  name="robot">
     <xacro:include filename="robot_core.xacro"/>
-    <xacro:include filename="gazebo_control.xacro"/>
+    <xacro:include filename="ros2_control.xacro"/>
+    <!-- <xacro:include filename="gazebo_control.xacro"/> -->
+    <xacro:include filename="lidar.xacro"/>
 </robot>

File: description/robot_core.xacro (robot description, xacro)
@@ -14,6 +14,17 @@
         <color rgba="0 0 0 1"/>
     </material>
+    <material name="red">
+        <color rgba="1 0 0 1"/>
+    </material>
     <!-- BASE LINK -->
     <link name="base_link">
+    </link>
+    <!-- BASE_FOOTPRINT LINK -->
+    <joint name="base_footprint_link" type="fixed">
+        <parent link="base_link"/>
+        <child link="base_footprint"/>
+        <origin xyz="0 0 0" rpy-="0 0 0"/>
+    </joint>
+    <link name="base_footprint">
     </link>
     <!-- CHASSIS LINK -->
@@ -37,5 +48,5 @@
             </geometry>
         </collision>
-        <xacro:inertial_box mass="10" x="0.58" y="0.3" z="0.34">
+        <xacro:inertial_box mass="7" x="0.58" y="0.3" z="0.34">
             <origin xyz="0.29 0 0.17" rpy="0 0 0"/>
         </xacro:inertial_box>
@@ -65,5 +76,5 @@
             <material name="white"/>
         </collision>
-        <xacro:inertial_box mass="1.5" x="0.25" y="0.26" z="0.145">
+        <xacro:inertial_box mass="0.5" x="0.25" y="0.26" z="0.145">
             <origin xyz="0 0 0.068" rpy="0 0 0"/>
         </xacro:inertial_box>
@@ -133,5 +144,5 @@
         <visual>
             <geometry>
-                <sphere radius="0.06"/>
+                <sphere radius="0.059"/>
             </geometry>
             <material name="black"/>
@@ -139,5 +150,5 @@
         <collision>
             <geometry>
-                <sphere radius="0.06"/>
+                <sphere radius="0.059"/>
             </geometry>
         </collision>
@@ -160,5 +171,5 @@
         <visual>
             <geometry>
-                <sphere radius="0.06"/>
+                <sphere radius="0.059"/>
             </geometry>
             <material name="black"/>
@@ -166,5 +177,5 @@
         <collision>
             <geometry>
-                <sphere radius="0.06"/>
+                <sphere radius="0.059"/>
             </geometry>
         </collision>

Commit message: trying to real robot working

File: description/robot.urdf.xacro (robot description, xacro)
@@ -1,7 +1,13 @@
 <?xml version="1.0"?>
 <robot xmlns:xacro="http://www.ros.org/wiki/xacro"  name="robot">
+    <xacro:arg name="use_ros2_control" default="true"/>
+    <xacro:arg name="sim_mode" default="false"/>
     <xacro:include filename="robot_core.xacro"/>
-    <xacro:include filename="ros2_control.xacro"/>
-    <!-- <xacro:include filename="gazebo_control.xacro"/> -->
+    <xacro:if value="$(arg use_ros2_control)">
+        <xacro:include filename="ros2_control.xacro"/>
+    </xacro:if>
+    <xacro:unless value="$(arg use_ros2_control)">
+        <xacro:include filename="gazebo_control.xacro"/>
+    </xacro:unless>
     <xacro:include filename="lidar.xacro"/>
 </robot>

File: description/ros2_control.xacro (robot description, xacro)
@@ -1,5 +1,60 @@
 <?xml version="1.0"?>
 <robot xmlns:xacro="http://www.ros.org/wiki/xacro">
-    <ros2_control name="GazeboSystem" type="system">
+    <!-- <ros2_control name="RealRobot" type="system">
+        <hardware>
+            <plugin>cmd_vel_to_arduino/CmdVelToArduino</plugin>
+            <param name='left_wheel_name'></param>
+            <param name='right_wheel_name'></param>
+            <param name='loop_rate'>30</param>
+            <param name='device'>/dev/ttyUSB0</param>
+            <param name='baud_rate'>115200</param>
+            <param name='timeout'>1000</param>
+        </hardware>
+        <joint name="left_wheel_joint">
+            <command_interface name="velocity">
+                <param name="min">-10</param>
+                <param name="max">10</param>
+            </command_interface>
+            <state_interface name="velocity"/>
+            <state_interface name="position"/>
+        </joint>
+        <joint name="right_wheel_joint">
+            <command_interface name="velocity">
+                <param name="min">-10</param>
+                <param name="max">10</param>
+            </command_interface>
+            <state_interface name="velocity"/>
+            <state_interface name="position"/>
+        </joint>
+    </ros2_control> -->
+    <!-- <ros2_control name="RealRobot" type="system">
+        <hardware>
+            <plugin>diffdrive_arduino/DiffDriveArduino</plugin>
+            <param name='left_wheel_name'>left_wheel_joint</param>
+            <param name='right_wheel_name'>right_wheel_joint</param>
+            <param name='loop_rate'>30</param>
+            <param name='device'>/dev/ttyUSB0</param>
+            <param name='baud_rate'>115200</param>
+            <param name='timeout'>1000</param>
+            <param name='enc_counts_per_rev'></param>
+        </hardware>
+        <joint name="left_wheel_joint">
+            <command_interface name="velocity">
+                <param name="min">-10</param>
+                <param name="max">10</param>
+            </command_interface>
+            <state_interface name="velocity"/>
+            <state_interface name="position"/>
+        </joint>
+        <joint name="right_wheel_joint">
+            <command_interface name="velocity">
+                <param name="min">-10</param>
+                <param name="max">10</param>
+            </command_interface>
+            <state_interface name="velocity"/>
+            <state_interface name="position"/>
+        </joint>
+    </ros2_control> -->
+    <!-- <ros2_control name="GazeboSystem" type="system">
         <hardware>
             <plugin>gazebo_ros2_control/GazeboSystem</plugin>
@@ -26,4 +81,63 @@
             <parameters>$(find art_amr)/config/amr_controllers.yaml</parameters>
         </plugin>
+    </gazebo> -->
+    <xacro:unless value="$(arg sim_mode)">
+        <ros2_control name="RealRobot" type="system">
+            <hardware>
+                <plugin>diffdrive_arduino/DiffDriveArduino</plugin>
+                <param name="left_wheel_name">left_wheel_joint</param>
+                <param name="right_wheel_name">right_wheel_joint</param>
+                <param name="loop_rate">30</param>
+                <param name="device">/dev/ttyUSB0</param>
+                <param name="baud_rate">115200</param>
+                <param name="timeout">1000</param>
+                <param name="enc_counts_per_rev">3436</param>
+            </hardware>
+            <joint name="left_wheel_joint">
+                <command_interface name="velocity">
+                    <param name="min">-10</param>
+                    <param name="max">10</param>
+                </command_interface>
+                <state_interface name="velocity"/>
+                <state_interface name="position"/>
+            </joint>
+            <joint name="right_wheel_joint">
+                <command_interface name="velocity">
+                    <param name="min">-10</param>
+                    <param name="max">10</param>
+                </command_interface>
+                <state_interface name="velocity"/>
+                <state_interface name="position"/>
+            </joint>
+        </ros2_control>
+    </xacro:unless>
+    <xacro:if value="$(arg sim_mode)">
+        <ros2_control name="GazeboSystem" type="system">
+            <hardware>
+                <plugin>gazebo_ros2_control/GazeboSystem</plugin>
+            </hardware>
+            <joint name="left_wheel_joint">
+                <command_interface name="velocity">
+                    <param name="min">-10</param>
+                    <param name="max">10</param>
+                </command_interface>
+                <state_interface name="velocity"/>
+                <state_interface name="position"/>
+            </joint>
+            <joint name="right_wheel_joint">
+                <command_interface name="velocity">
+                    <param name="min">-10</param>
+                    <param name="max">10</param>
+                </command_interface>
+                <state_interface name="velocity"/>
+                <state_interface name="position"/>
+            </joint>
+        </ros2_control>
+    </xacro:if>
+    <gazebo>
+        <plugin name="gazebo_ros2_control" filename="libgazebo_ros2_control.so">
+            <parameters>$(find art_amr)/config/amr_controllers.yaml</parameters>
+            <parameters>$(find art_amr)/config/gaz_ros2_ctl_use_sim.yaml</parameters>
+        </plugin>
     </gazebo>
 </robot>
