Commit message: Edit robot.launch +  some stuff.

File: description/lidar.xacro (robot description, xacro)
@@ -2,7 +2,7 @@
 <robot xmlns:xacro="http://www.ros.org/wiki/xacro" >
     <joint name="laser_joint" type="fixed">
-        <parent link="chassis"/>
+        <parent link="base_link"/>
         <child link="laser_frame"/>
-        <origin xyz="0.5 0 0.36" rpy="0 0 0"/>
+        <origin xyz="0.25 0 0.36" rpy="0 0 0"/>
     </joint>
     <link name="laser_frame">

File: description/ros2_control.xacro (robot description, xacro)
@@ -92,5 +92,5 @@
                 <param name="baud_rate">115200</param>
                 <param name="timeout_ms">1000</param>
-                <param name="enc_counts_per_rev">12700</param>
+                <param name="enc_counts_per_rev">4350</param>
             </hardware>
             <joint name="left_wheel_joint">

Commit message: Add files via upload

File: description/lidar.xacro (robot description, xacro)
@@ -3,6 +3,8 @@
     <joint name="laser_joint" type="fixed">
         <parent link="base_link"/>
+        <!-- <parent link="chassis"/> -->
         <child link="laser_frame"/>
         <origin xyz="0.25 0 0.36" rpy="0 0 0"/>
+        <!-- <origin xyz="0.55 0 0.36" rpy="0 0 0"/> -->
     </joint>
     <link name="laser_frame">

File: description/ros2_control.xacro (robot description, xacro)
@@ -88,9 +88,9 @@
                 <param name="left_wheel_name">left_wheel_joint</param>
                 <param name="right_wheel_name">right_wheel_joint</param>
-                <param name="loop_rate">10</param>
+                <param name="loop_rate">30</param>
                 <param name="device">/dev/ttyUSB0</param>
                 <param name="baud_rate">115200</param>
                 <param name="timeout_ms">1000</param>
-                <param name="enc_counts_per_rev">4350</param>
+                <param name="enc_counts_per_rev">3450</param>
             </hardware>
             <joint name="left_wheel_joint">
